File: E103-RTL8812CU-Breakout-Board.kicad_pcb (KiCad board)
At the start: 4 copper layers, 47.5 x 50.7 mm, 20 parts, among them J1 USB_C_Receptacle_USB2.0_16P, J2 USB_C_Receptacle_USB2.0_16P, U1 Buck_Converter_3.3V, U2 E103-RTL8812CU

Commit message: boards ordered
Parts:
- removed J1: USB_C_Receptacle_USB2.0_16P, Connector_USB:USB_C_Receptacle_GCT_USB4105-xx-A_16P_TopMnt_Horizontal
- removed R1, R5: 5.1k, Resistor_SMD:R_0805_2012Metric
- added C5: 47u, Capacitor_THT:CP_Radial_D5.0mm_P2.00mm, F.Cu at (138.5, 97.5)
- added C6: 47u, Capacitor_THT:CP_Radial_D5.0mm_P2.00mm, F.Cu at (150.0, 121.5)
- added D1: VS-10BQ015-M3, Diode_SMD:D_SMB_Handsoldering, F.Cu at (116.5, 120.0)
- R3, R4: footprint Resistor_SMD:R_0805_2012Metric -> Resistor_SMD:R_0402_1005Metric
- TP1, TP2, TP3, TP4: moved to B.Cu
- moved C1 5.80 mm to (157.0, 115.8)
- moved C2 5.80 mm to (152.0, 86.3)
- moved TP5 5.80 mm to (147.5, 86.3)
- moved TP6 5.80 mm to (156.5, 86.3)
- moved U1 5.80 mm to (152.0, 100.8)
- moved R4 0.40 mm to (129.5, 114.4)
- turned TP1 to 180 degrees
- turned TP2 to 180 degrees
- turned TP3 to 180 degrees
- turned TP4 to 180 degrees
Connections:
- R2 pad 1: /V_IN -> Net-(D1-A)
Routing:
- net GND: track 16.3 -> 39.2 mm, vias 56 -> 57
- net +3.3V: track 3.92 -> 11.3 mm, vias 16 -> 17
- net Net-(J1-CC1): track 4.72 -> 0.00 mm
- net /V_IN: track 3.57 -> 0.00 mm, vias 15 -> 10
- net Net-(J1-CC2): track 3.51 -> 0.00 mm
- net Net-(J2-VBUS-PadA4): track 3.11 -> 0.00 mm, vias 4 -> 0
- added copper zone on F.Cu, net Net-(D1-A)
Other:
- outline, holes or cut-outs redrawn
- board text added: "+5V"
- board text added: "3.3V"
- board text added: "5-30V → 3.3V"
- board text added: "DATA"
- board text added: "GND"
- board text added: "RESET"
